Commit message: Manual Control & Sensors

File: src/auto_drive/urdf/my_car.urdf (robot description, URDF)
Before this commit: robot my_car, 11 links, 10 joints
Links:
- added link lidar_link, mass 0.05; visual cylinder length=0.03 radius=0.02
Joints:
- added joint lidar_joint: type fixed, parent base_link, child lidar_link, origin xyz=0 0 0.08 rpy=0 0 0
